File: hardware/hack_soc_shield/hack_soc_shield.kicad_pcb (KiCad board)
At the start: 2 copper layers, 76.2 x 73.8 mm, 27 parts, among them J1 Conn_01x05_Pin, J10 Conn_01x27_Female, J11 Conn_01x20_Female, J2 Conn_01x10_Pin, J5 Conn_01x05_Pin, SW1 SW_Push, SW2 SW_DIP_x02, U1 23LC1024, U2 23LC1024, U3 23LC1024

Commit message: Update hack_soc_shield
Parts:
- added SW3: SW_DIP_x02, Button_Switch_THT:SW_DIP_SPSTx03_Slide_9.78x9.8mm_W7.62mm_P2.54mm, F.Cu at (83.2, 88.9)
Connections:
- R1 pad 2: mprj_io[8] -> ram_cs
- R2 pad 2: mprj_io[14] -> rom_cs
- R3 pad 2: mprj_io[20] -> vram_cs
- U1 pad 1: mprj_io[8] -> ram_cs
- U2 pad 1: mprj_io[14] -> rom_cs
- U3 pad 1: mprj_io[20] -> vram_cs
Routing:
- net vram_cs: track 0.00 -> 63.9 mm
- net ram_cs: track 0.00 -> 40.1 mm
- net rom_cs: track 0.00 -> 37.5 mm
- net mprj_io[14]: track 38.1 -> 59.1 mm
- net mprj_io[20]: track 37.6 -> 54.2 mm
- net mprj_io[8]: track 37.7 -> 32.0 mm
- net +3.3V: track 230.5 -> 228.3 mm, vias 1 -> 2
Other:
- board text added: "Hack SoC Shield v0.1"
- board text added: "SRAM toggle"
- board text removed: "Hack SoC Shileld"

Commit message: Update hardware
Routing:
- net mprj_io[29]: track 17.3 -> 16.6 mm
- net GND: vias 9 -> 10
Other:
- board text added: "3.3v"
- board text added: "hsync"
- board text added: "rgb"
- board text added: "vsync"
